File: 1819-hardware/Autopilot/Autopilot.brd (EAGLE design)
At the start: 44.4 x 54 mm, 36 parts, among them U1 PCA9615, U3 74HC1G04, U4 MAX3485CSA, U5 V_REG_LD1117VXXLD1117-SMD

Commit message: worked on boards
Connections:
- net 3V3: now also U2.1; no longer U2.2
- net GND: now also U2.4; no longer U2.1
- net SCL3V3: now also U2.2; no longer U2.3
- net SDA3V3: now also U2.3; no longer U2.4
